Commit message: Changed some friction parameters

File: minitaur_description/urdf/minitaur_gazebo.urdf.xacro (robot description, xacro)
@@ -62,5 +62,5 @@
 	<xacro:property name="toeDamping" value="1000.0"/>
 	<xacro:property name="toeSpinningFriction" value="1.0"/>
-	<xacro:property name="toeLateralFriction" value="70"/>
+	<xacro:property name="toeLateralFriction" value="1.0"/>
 	<!-- LINK: Body dummy -->
 	<link name="base_chassis_link_dummy">
